File: Electrónica/horno_reflujo/horno_reflujo.kicad_sch (KiCad schematic)
At the start: 42 parts, among them J1 LevelShifter, J10 ssr1, J11 ssr2, J12 encoder, J13 Max6675_modulo2, J14 Max6675_modulo3, J15 Max6675_modulo4, J2 LevelShifter, J3 Display Oled I2C, J4 Max6675_modulo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

Commit message: actualización del main
Parts:
- removed F3: 15A, Fuse:Fuseholder_Cylinder-5x20mm_Schurter_0031_8201_Horizontal_Open, symbol PCM_Device_AKL:Fuse
- removed J9: resistencia1, Connector_PinHeader_2.54mm:PinHeader_1x01_P2.54mm_Vertical, symbol Connector:Conn_01x01_Pin
- removed U3: 74LS14, symbol 74xx:74LS14
- removed U4: LM7833CT, Package_TO_SOT_THT:TO-220-3_Vertical, symbol PCM_Voltage_Regulator_AKL:LM7805CT
- added R11, R8, R9: 10K, Resistor_THT:R_Axial_DIN0207_L6.3mm_D2.5mm_P2.54mm_Vertical, symbol Device:R_US
- added U1: LD1117S33TR_SOT223, Package_TO_SOT_SMD:SOT-223-3_TabPin2, symbol Regulator_Linear:LD1117S33TR_SOT223
- added U2: 74LS14, Package_DIP:DIP-14_W7.62mm_Socket_LongPads, symbol 74xx:74LS14
- H1, H2, H3, H4: footprint MountingHole:MountingHole_2.2mm_M2_DIN965 -> MountingHole:MountingHole_3.2mm_M3_DIN965
- J10, J11, J6, J7: footprint TerminalBlock:TerminalBlock_Xinya_XY308-2.54-2P_1x02_P2.54mm_Horizontal -> TerminalBlock:TerminalBlock_bornier-2_P5.08mm
- R10, R7: footprint Resistor_THT:R_Axial_DIN0204_L3.6mm_D1.6mm_P7.62mm_Horizontal -> Resistor_THT:R_Axial_DIN0207_L6.3mm_D2.5mm_P2.54mm_Vertical
- R5, R6: footprint Resistor_THT:R_Axial_DIN0411_L9.9mm_D3.6mm_P15.24mm_Horizontal -> Resistor_THT:R_Axial_DIN0411_L9.9mm_D3.6mm_P5.08mm_Vertical
Connections:
- net +3.3V: now also U1.2 (VO); no longer J13.2 (Pin_2), J14.2 (Pin_2), J15.2 (Pin_2), J4.2 (Pin_2)
- net +5V: now also R11.2, R8.2, R9.2, U1.3 (VI), U2.14 (VCC)
- net ENCODER_A: now also R8.1
- net ENCODER_B: now also R9.1
- net ENCODER_BTN: now also R11.1
- net GND: now also U1.1 (GND), U2.7 (GND)
- net LINE: now also J6.2 (Pin_2), J7.2 (Pin_2); no longer J6.1 (Pin_1), R5.2
- net NEUT: now also J6.1 (Pin_1); no longer J6.2 (Pin_2), J7.2 (Pin_2)
- net fan: now also U2.3
- net fire: now also U2.5
- net zero: now also U2.2
- net +3.3Vmc: now reaches dev_board1.38 (3.3)
- net +3.3Vmc: now also J13.2 (Pin_2), J14.2 (Pin_2), J15.2 (Pin_2), J4.2 (Pin_2)
- net at J10.1 (Pin_1): now also U2.6
- net at F2.2, J8.1 (Pin_1): now also R5.2
- net at OC1.4, R7.1: now also U2.1
- net at R10.2: now also U2.4
- no-connect marks 6 -> 11
Other:
- moved on the sheet: C5
